Commit message: something bad has happen

File: src/four_wheel_drive/robot_model/xacro/smartcar_sim.xacro (robot description, xacro)
@@ -151,51 +151,4 @@
 		</sensor>
 	</gazebo>
-    <!-- Drive controller -->
-<!--	<gazebo>
-		<plugin name="skid_steer_drive_controller" filename="libgazebo_ros_skid_steer_drive.so">
-			<updateRate>100.0</updateRate>
-			<robotNamespace></robotNamespace>
-			<leftFrontJoint>left_front_wheel_joint</leftFrontJoint>
-			<rightFrontJoint>right_front_wheel_joint</rightFrontJoint>
-			<leftRearJoint>left_back_wheel_joint</leftRearJoint>
-			<rightRearJoint>right_back_wheel_joint</rightRearJoint>
-			<wheelSeparation>0.16</wheelSeparation>
-			<wheelDiameter>0.05</wheelDiameter>
-			<commandTopic>cmd_vel</commandTopic>
-			<odometryTopic>odom</odometryTopic>
-			<robotBaseFrame>base_footprint</robotBaseFrame>
-			<odometryFrame>odom</odometryFrame>
-			<torque>15</torque>
-			<topicName>cmd_vel</topicName>
-			<broadcastTF>1</broadcastTF>
-	  	</plugin>
-	</gazebo>
--->
-<!--
-	<gazebo>
-            <plugin name="differential_drive_controller"
-                    filename="libgazebo_ros_diff_drive.so">
-                <rosDebugLevel>Debug</rosDebugLevel>
-                <publishWheelTF>true</publishWheelTF>
-                <robotNamespace>/</robotNamespace>
-                <publishTf>1</publishTf>
-                <publishWheelJointState>true</publishWheelJointState>
-                <alwaysOn>true</alwaysOn>
-                <updateRate>100.0</updateRate>
-                <legacyMode>true</legacyMode>
-                <leftJoint>left_back_wheel_joint</leftJoint>
-                <rightJoint>right_back_wheel_joint</rightJoint>
-                <wheelSeparation>0.16</wheelSeparation>
-                <wheelDiameter>0.05</wheelDiameter>
-                <broadcastTF>1</broadcastTF>
-                <wheelTorque>20</wheelTorque>
-                <wheelAcceleration>1.8</wheelAcceleration>
-                <commandTopic>cmd_vel</commandTopic>
-                <odometryFrame>odom</odometryFrame>
-                <odometryTopic>odom</odometryTopic>
-                <robotBaseFrame>base_footprint</robotBaseFrame>
-            </plugin>
-        </gazebo>
--->
 	<!-- Transmission is important to link the joints and the controller -->
 	<transmission name="right_bridge_joint_trans">
@@ -213,13 +166,32 @@
 		<type>transmission_interface/SimpleTransmission</type>
 		<joint name="left_bridge_to_bridge" >
-			<hardwareInterface>hardware_interface/EffortJointInterface</hardwareInterface>
+			<hardwareInterface>hardware_interface/PositionJointInterface</hardwareInterface>
 		</joint>
 		<actuator name="left_bridge_joint_motor">
-			<hardwareInterface>hardware_interface/EffortJointInterface</hardwareInterface>
+			<hardwareInterface>hardware_interface/PositionJointInterface</hardwareInterface>
 			<mechanicalReduction>1</mechanicalReduction>
 			<motorTorqueConstant>100</motorTorqueConstant>
 		</actuator>
 	</transmission>
-<!--
+	<transmission name="right_back_wheel_joint_trans">
+		<type>transmission_interface/SimpleTransmission</type>
+		<joint name="right_back_wheel_joint" >
+			<hardwareInterface>hardware_interface/VelocityJointInterface</hardwareInterface>
+		</joint>
+		<actuator name="right_back_wheel_joint_motor">
+			<hardwareInterface>hardware_interface/VelocityJointInterface</hardwareInterface>
+			<mechanicalReduction>1</mechanicalReduction>
+		</actuator>
+	</transmission>
+	<transmission name="left_back_wheel_joint_trans">
+		<type>transmission_interface/SimpleTransmission</type>
+		<joint name="left_back_wheel_joint" >
+			<hardwareInterface>hardware_interface/VelocityJointInterface</hardwareInterface>
+		</joint>
+		<actuator name="left_back_wheel_joint_motor">
+			<hardwareInterface>hardware_interface/VelocityJointInterface</hardwareInterface>
+			<mechanicalReduction>1</mechanicalReduction>
+		</actuator>
+	</transmission>
 	<transmission name="right_front_wheel_joint_trans">
 		<type>transmission_interface/SimpleTransmission</type>
@@ -242,64 +214,4 @@
 		</actuator>
 	</transmission>
--->
-	<transmission name="right_back_wheel_joint_trans">
-		<type>transmission_interface/SimpleTransmission</type>
-		<joint name="right_back_wheel_joint" >
-			<hardwareInterface>hardware_interface/VelocityJointInterface</hardwareInterface>
-		</joint>
-		<actuator name="right_back_wheel_joint_motor">
-			<hardwareInterface>hardware_interface/VelocityJointInterface</hardwareInterface>
-			<mechanicalReduction>1</mechanicalReduction>
-		</actuator>
-	</transmission>
-	<transmission name="left_back_wheel_joint_trans">
-		<type>transmission_interface/SimpleTransmission</type>
-		<joint name="left_back_wheel_joint" >
-			<hardwareInterface>hardware_interface/VelocityJointInterface</hardwareInterface>
-		</joint>
-		<actuator name="left_back_wheel_joint_motor">
-			<hardwareInterface>hardware_interface/VelocityJointInterface</hardwareInterface>
-			<mechanicalReduction>1</mechanicalReduction>
-		</actuator>
-	</transmission>
-	<transmission name="right_front_wheel_joint_trans">
-		<type>transmission_interface/SimpleTransmission</type>
-		<joint name="right_front_wheel_to_bridge" >
-			<hardwareInterface>hardware_interface/VelocityJointInterface</hardwareInterface>
-		</joint>
-		<actuator name="right_front_wheel_joint_motor">
-			<hardwareInterface>hardware_interface/VelocityJointInterface</hardwareInterface>
-			<mechanicalReduction>1</mechanicalReduction>
-		</actuator>
-	</transmission>
-	<transmission name="left_front_wheel_joint_trans">
-		<type>transmission_interface/SimpleTransmission</type>
-		<joint name="left_front_wheel_to_bridge" >
-			<hardwareInterface>hardware_interface/VelocityJointInterface</hardwareInterface>
-		</joint>
-		<actuator name="left_front_wheel_joint_motor">
-			<hardwareInterface>hardware_interface/VelocityJointInterface</hardwareInterface>
-			<mechanicalReduction>1</mechanicalReduction>
-		</actuator>
-	</transmission>
-	<!-- Friction Parametres -->
-<!--
-	<gazebo reference="left_bridge">
-		<mu1>10000000000000</mu1>
-		<mu2>10000000000000</mu2>
-		<kp>100000000</kp>
-		<kd>1</kd>
-		<minDepth>0.01</minDepth>
-		<maxVel>101</maxVel>
-	</gazebo>
-	<gazebo reference="right_bridge">
-		<mu1>10000000000000</mu1>
-		<mu2>10000000000000</mu2>
-		<kp>100000000</kp>
-		<kd>1</kd>
-		<minDepth>0.01</minDepth>
-		<maxVel>100</maxVel>
-	</gazebo>
--->
 	<gazebo reference="right_back_wheel">
 		<mu1>10000000000000</mu1>
